File: Projects/Wemos test/Wemos Test.kicad_pcb (KiCad board)
At the start: 2 copper layers, 1 part, among them U1 wemos_mini_wide

Commit message: Added notes to Build info for Sonoff switch
Parts:
- U1: value wemos_mini_wide -> Wemos_D1_Mini_wide
Connections:
- U1 pad 1: Net-(U1-Pad1) -> (no net)
- U1 pad 10: Net-(U1-Pad10) -> (no net)
- U1 pad 11: Net-(U1-Pad11) -> (no net)
- U1 pad 12: Net-(U1-Pad12) -> (no net)
- U1 pad 13: Net-(U1-Pad13) -> (no net)
- U1 pad 14: Net-(U1-Pad14) -> (no net)
- U1 pad 15: Net-(U1-Pad15) -> (no net)
- U1 pad 16: Net-(U1-Pad16) -> (no net)
- U1 pad 2: Net-(U1-Pad2) -> (no net)
- U1 pad 3: Net-(U1-Pad3) -> (no net)
- U1 pad 4: Net-(U1-Pad4) -> (no net)
- U1 pad 5: Net-(U1-Pad5) -> (no net)
- U1 pad 6: Net-(U1-Pad6) -> (no net)
- U1 pad 7: Net-(U1-Pad7) -> (no net)
- U1 pad 8: Net-(U1-Pad8) -> (no net)
- U1 pad 9: Net-(U1-Pad9) -> (no net)
Changed lines of the file:
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@@
     (zones 0)
     (modules 1)
-    (nets 17)
+    (nets 1)
   )
   (page A4)
@@
   )
   (net 0 "")
-  (net 1 "Net-(U1-Pad8)")
-  (net 2 "Net-(U1-Pad7)")
-  (net 3 "Net-(U1-Pad6)")
-  (net 4 "Net-(U1-Pad5)")
-  (net 5 "Net-(U1-Pad4)")
-  (net 6 "Net-(U1-Pad3)")
-  (net 7 "Net-(U1-Pad2)")
-  (net 8 "Net-(U1-Pad1)")
-  (net 9 "Net-(U1-Pad16)")
-  (net 10 "Net-(U1-Pad15)")
-  (net 11 "Net-(U1-Pad14)")
-  (net 12 "Net-(U1-Pad13)")
-  (net 13 "Net-(U1-Pad12)")
-  (net 14 "Net-(U1-Pad11)")
-  (net 15 "Net-(U1-Pad10)")
-  (net 16 "Net-(U1-Pad9)")
   (net_class Default "This is the default net class."
     (clearance 0.2)
@@
     (uvia_dia 0.3)
     (uvia_drill 0.1)
-    (add_net "Net-(U1-Pad1)")
-    (add_net "Net-(U1-Pad10)")
-    (add_net "Net-(U1-Pad11)")
-    (add_net "Net-(U1-Pad12)")
-    (add_net "Net-(U1-Pad13)")
-    (add_net "Net-(U1-Pad14)")
-    (add_net "Net-(U1-Pad15)")
-    (add_net "Net-(U1-Pad16)")
-    (add_net "Net-(U1-Pad2)")
-    (add_net "Net-(U1-Pad3)")
-    (add_net "Net-(U1-Pad4)")
-    (add_net "Net-(U1-Pad5)")
-    (add_net "Net-(U1-Pad6)")
-    (add_net "Net-(U1-Pad7)")
-    (add_net "Net-(U1-Pad8)")
-    (add_net "Net-(U1-Pad9)")
   )
   (module My_Component_Footprints:Wemos_D1_mini_board (layer F.Cu)
@@
       (effects (font (size 1 1) (thickness 0.15)))
     )
-    (fp_text value wemos_mini_wide (at 1.27 -19.05) (layer F.Fab)
+    (fp_text value Wemos_D1_Mini_wide (at 1.27 -19.05) (layer F.Fab)
       (effects (font (size 1 1) (thickness 0.15)))
     )
@@
       (effects (font (size 3 3) (thickness 0.15)))
     )
-    (pad 9 thru_hole circle (at 11.43 -10.16) (size 1.8 1.8) (drill 1.016) (layers *.Cu *.Mask F.SilkS)
-      (net 16 "Net-(U1-Pad9)"))
-    (pad 10 thru_hole circle (at 11.43 -7.62) (size 1.8 1.8) (drill 1.016) (layers *.Cu *.Mask F.SilkS)
-      (net 15 "Net-(U1-Pad10)"))
-    (pad 11 thru_hole circle (at 11.43 -5.08) (size 1.8 1.8) (drill 1.016) (layers *.Cu *.Mask F.SilkS)
-      (net 14 "Net-(U1-Pad11)"))
-    (pad 12 thru_hole circle (at 11.43 -2.54) (size 1.8 1.8) (drill 1.016) (layers *.Cu *.Mask F.SilkS)
-      (net 13 "Net-(U1-Pad12)"))
-    (pad 13 thru_hole circle (at 11.43 0) (size 1.8 1.8) (drill 1.016) (layers *.Cu *.Mask F.SilkS)
-      (net 12 "Net-(U1-Pad13)"))
-    (pad 14 thru_hole circle (at 11.43 2.54) (size 1.8 1.8) (drill 1.016) (layers *.Cu *.Mask F.SilkS)
-      (net 11 "Net-(U1-Pad14)"))
-    (pad 15 thru_hole circle (at 11.43 5.08) (size 1.8 1.8) (drill 1.016) (layers *.Cu *.Mask F.SilkS)
-      (net 10 "Net-(U1-Pad15)"))
-    (pad 16 thru_hole circle (at 11.43 7.62) (size 1.8 1.8) (drill 1.016) (layers *.Cu *.Mask F.SilkS)
-      (net 9 "Net-(U1-Pad16)"))
-    (pad 1 thru_hole circle (at -11.43 7.62) (size 1.8 1.8) (drill 1.016) (layers *.Cu *.Mask F.SilkS)
-      (net 8 "Net-(U1-Pad1)"))
-    (pad 2 thru_hole circle (at -11.43 5.08) (size 1.8 1.8) (drill 1.016) (layers *.Cu *.Mask F.SilkS)
-      (net 7 "Net-(U1-Pad2)"))
-    (pad 3 thru_hole circle (at -11.43 2.54) (size 1.8 1.8) (drill 1.016) (layers *.Cu *.Mask F.SilkS)
-      (net 6 "Net-(U1-Pad3)"))
-    (pad 4 thru_hole circle (at -11.43 0) (size 1.8 1.8) (drill 1.016) (layers *.Cu *.Mask F.SilkS)
-      (net 5 "Net-(U1-Pad4)"))
-    (pad 5 thru_hole circle (at -11.43 -2.54) (size 1.8 1.8) (drill 1.016) (layers *.Cu *.Mask F.SilkS)
-      (net 4 "Net-(U1-Pad5)"))
-    (pad 6 thru_hole circle (at -11.43 -5.08) (size 1.8 1.8) (drill 1.016) (layers *.Cu *.Mask F.SilkS)
-      (net 3 "Net-(U1-Pad6)"))
-    (pad 7 thru_hole circle (at -11.43 -7.62) (size 1.8 1.8) (drill 1.016) (layers *.Cu *.Mask F.SilkS)
-      (net 2 "Net-(U1-Pad7)"))
-    (pad 8 thru_hole circle (at -11.43 -10.16) (size 1.8 1.8) (drill 1.016) (layers *.Cu *.Mask F.SilkS)
-      (net 1 "Net-(U1-Pad8)"))
+    (pad 9 thru_hole circle (at 11.43 -10.16) (size 1.8 1.8) (drill 1.016) (layers *.Cu *.Mask F.SilkS))
+    (pad 10 thru_hole circle (at 11.43 -7.62) (size 1.8 1.8) (drill 1.016) (layers *.Cu *.Mask F.SilkS))
+    (pad 11 thru_hole circle (at 11.43 -5.08) (size 1.8 1.8) (drill 1.016) (layers *.Cu *.Mask F.SilkS))
+    (pad 12 thru_hole circle (at 11.43 -2.54) (size 1.8 1.8) (drill 1.016) (layers *.Cu *.Mask F.SilkS))
+    (pad 13 thru_hole circle (at 11.43 0) (size 1.8 1.8) (drill 1.016) (layers *.Cu *.Mask F.SilkS))
+    (pad 14 thru_hole circle (at 11.43 2.54) (size 1.8 1.8) (drill 1.016) (layers *.Cu *.Mask F.SilkS))
+    (pad 15 thru_hole circle (at 11.43 5.08) (size 1.8 1.8) (drill 1.016) (layers *.Cu *.Mask F.SilkS))
+    (pad 16 thru_hole circle (at 11.43 7.62) (size 1.8 1.8) (drill 1.016) (layers *.Cu *.Mask F.SilkS))
+    (pad 1 thru_hole circle (at -11.43 7.62) (size 1.8 1.8) (drill 1.016) (layers *.Cu *.Mask F.SilkS))
+    (pad 2 thru_hole circle (at -11.43 5.08) (size 1.8 1.8) (drill 1.016) (layers *.Cu *.Mask F.SilkS))
+    (pad 3 thru_hole circle (at -11.43 2.54) (size 1.8 1.8) (drill 1.016) (layers *.Cu *.Mask F.SilkS))
+    (pad 4 thru_hole circle (at -11.43 0) (size 1.8 1.8) (drill 1.016) (layers *.Cu *.Mask F.SilkS))
+    (pad 5 thru_hole circle (at -11.43 -2.54) (size 1.8 1.8) (drill 1.016) (layers *.Cu *.Mask F.SilkS))
+    (pad 6 thru_hole circle (at -11.43 -5.08) (size 1.8 1.8) (drill 1.016) (layers *.Cu *.Mask F.SilkS))
+    (pad 7 thru_hole circle (at -11.43 -7.62) (size 1.8 1.8) (drill 1.016) (layers *.Cu *.Mask F.SilkS))
+    (pad 8 thru_hole circle (at -11.43 -10.16) (size 1.8 1.8) (drill 1.016) (layers *.Cu *.Mask F.SilkS))
   )
 )
