File: Projects/Wemos test/Wemos Test.sch (KiCad schematic (older format))
At the start: 2 parts, among them U1 Wemos_D1_Mini_wide

Commit message: Added notes to Build info for Sonoff switch
Parts:
- U1: footprint (none) -> My_Component_Footprints:Wemos_D1_mini_board
Changed lines of the file:
@@
 EESchema Schematic File Version 4
+LIBS:Wemos Test-cache
 EELAYER 26 0
 EELAYER END
@@
 F 0 "U1" H 5000 3950 60  0000 C CNN
 F 1 "Wemos_D1_Mini_wide" H 5400 2850 60  0000 C CNN
-F 2 "" H 5750 2700 60  0000 C CNN
+F 2 "My_Component_Footprints:Wemos_D1_mini_board" H 5750 2700 60  0000 C CNN
 F 3 "" H 5750 2700 60  0000 C CNN
 	1    5200 3400
