File: Projects/Sonoff_4Ch_Switch/Relays.sch (KiCad schematic (older format))
At the start: 36 parts, among them K1 G5LE-1, K2 G5LE-1, K3 G5LE-1, K4 G5LE-1, Q1 2N7002, Q2 2N7002, Q3 2N7002, Q4 2N7002, Q5 2N7002, Q6 2N7002, Q7 2N7002, Q8 2N7002

Commit message: On to rev A2 of the 4 ch switch....
Parts:
- D5, D6, D7, D8: footprint LEDs:LED_0603_HandSoldering -> LEDs:LED_0805_HandSoldering
- R1, R10, R11, R12, R13, R14, R15, R16, R2, R3, R4, R5, R6, R7, R8, R9: footprint Resistor_SMD:R_0603_1608Metric_Pad1.05x0.95mm_HandSolder -> Resistors_SMD:R_0805_HandSoldering
Changed lines of the file:
@@
 EESchema Schematic File Version 4
-LIBS:Sonoff_4ch_switch-cache
 EELAYER 26 0
 EELAYER END
 $Descr A4 11693 8268
 encoding utf-8
-Sheet 2 3
-Title ""
+Sheet 2 2
+Title "Tasmota 4 Ch Switch - Relays and LED's"
 Date ""
-Rev ""
+Rev "1.0"
 Comp ""
 Comment1 ""
@@
 F 0 "R1" V 1493 2150 50  0000 C CNN
 F 1 "1K" V 1584 2150 50  0000 C CNN
-F 2 "Resistor_SMD:R_0603_1608Metric_Pad1.05x0.95mm_HandSolder" V 1630 2150 50  0001 C CNN
+F 2 "Resistors_SMD:R_0805_HandSoldering" V 1630 2150 50  0001 C CNN
 F 3 "~" H 1700 2150 50  0001 C CNN
 	1    1700 2150
@@
 F 0 "R2" H 1880 2354 50  0000 R CNN
 F 1 "10K" H 1880 2445 50  0000 R CNN
-F 2 "Resistor_SMD:R_0603_1608Metric_Pad1.05x0.95mm_HandSolder" V 1880 2400 50  0001 C CNN
+F 2 "Resistors_SMD:R_0805_HandSoldering" V 1880 2400 50  0001 C CNN
 F 3 "~" H 1950 2400 50  0001 C CNN
 	1    1950 2400
@@
 F 0 "R3" V 2343 3550 50  0000 C CNN
 F 1 "1K" V 2434 3550 50  0000 C CNN
-F 2 "Resistor_SMD:R_0603_1608Metric_Pad1.05x0.95mm_HandSolder" V 2480 3550 50  0001 C CNN
+F 2 "Resistors_SMD:R_0805_HandSoldering" V 2480 3550 50  0001 C CNN
 F 3 "~" H 2550 3550 50  0001 C CNN
 	1    2550 3550
@@
 F 0 "R4" H 2730 3754 50  0000 R CNN
 F 1 "10K" H 2730 3845 50  0000 R CNN
-F 2 "Resistor_SMD:R_0603_1608Metric_Pad1.05x0.95mm_HandSolder" V 2730 3800 50  0001 C CNN
+F 2 "Resistors_SMD:R_0805_HandSoldering" V 2730 3800 50  0001 C CNN
 F 3 "~" H 2800 3800 50  0001 C CNN
 	1    2800 3800
@@
 F 0 "R5" V 3343 4800 50  0000 C CNN
 F 1 "1K" V 3434 4800 50  0000 C CNN
-F 2 "Resistor_SMD:R_0603_1608Metric_Pad1.05x0.95mm_HandSolder" V 3480 4800 50  0001 C CNN
+F 2 "Resistors_SMD:R_0805_HandSoldering" V 3480 4800 50  0001 C CNN
 F 3 "~" H 3550 4800 50  0001 C CNN
 	1    3550 4800
@@
 F 0 "R6" H 3730 5004 50  0000 R CNN
 F 1 "10K" H 3730 5095 50  0000 R CNN
-F 2 "Resistor_SMD:R_0603_1608Metric_Pad1.05x0.95mm_HandSolder" V 3730 5050 50  0001 C CNN
+F 2 "Resistors_SMD:R_0805_HandSoldering" V 3730 5050 50  0001 C CNN
 F 3 "~" H 3800 5050 50  0001 C CNN
 	1    3800 5050
@@
 F 0 "R7" V 4343 6200 50  0000 C CNN
 F 1 "1K" V 4434 6200 50  0000 C CNN
-F 2 "Resistor_SMD:R_0603_1608Metric_Pad1.05x0.95mm_HandSolder" V 4480 6200 50  0001 C CNN
+F 2 "Resistors_SMD:R_0805_HandSoldering" V 4480 6200 50  0001 C CNN
 F 3 "~" H 4550 6200 50  0001 C CNN
 	1    4550 6200
@@
 F 0 "R8" H 4730 6404 50  0000 R CNN
 F 1 "10K" H 4730 6495 50  0000 R CNN
-F 2 "Resistor_SMD:R_0603_1608Metric_Pad1.05x0.95mm_HandSolder" V 4730 6450 50  0001 C CNN
+F 2 "Resistors_SMD:R_0805_HandSoldering" V 4730 6450 50  0001 C CNN
 F 3 "~" H 4800 6450 50  0001 C CNN
 	1    4800 6450
@@
 F 0 "R9" V 5943 2100 50  0000 C CNN
 F 1 "1K" V 6034 2100 50  0000 C CNN
-F 2 "Resistor_SMD:R_0603_1608Metric_Pad1.05x0.95mm_HandSolder" V 6080 2100 50  0001 C CNN
+F 2 "Resistors_SMD:R_0805_HandSoldering" V 6080 2100 50  0001 C CNN
 F 3 "~" H 6150 2100 50  0001 C CNN
 	1    6150 2100
@@
 F 0 "D5" V 6638 1233 50  0000 R CNN
 F 1 "LED" V 6547 1233 50  0000 R CNN
-F 2 "LEDs:LED_0603_HandSoldering" H 6600 1350 50  0001 C CNN
+F 2 "LEDs:LED_0805_HandSoldering" H 6600 1350 50  0001 C CNN
 F 3 "~" H 6600 1350 50  0001 C CNN
 	1    6600 1350
@@
 F 0 "R10" V 6393 1650 50  0000 C CNN
 F 1 "1K" V 6484 1650 50  0000 C CNN
-F 2 "Resistor_SMD:R_0603_1608Metric_Pad1.05x0.95mm_HandSolder" V 6530 1650 50  0001 C CNN
+F 2 "Resistors_SMD:R_0805_HandSoldering" V 6530 1650 50  0001 C CNN
 F 3 "~" H 6600 1650 50  0001 C CNN
 	1    6600 1650
@@
 F 0 "R11" V 6843 2950 50  0000 C CNN
 F 1 "1K" V 6934 2950 50  0000 C CNN
-F 2 "Resistor_SMD:R_0603_1608Metric_Pad1.05x0.95mm_HandSolder" V 6980 2950 50  0001 C CNN
+F 2 "Resistors_SMD:R_0805_HandSoldering" V 6980 2950 50  0001 C CNN
 F 3 "~" H 7050 2950 50  0001 C CNN
 	1    7050 2950
@@
 F 0 "D6" V 7538 2083 50  0000 R CNN
 F 1 "LED" V 7447 2083 50  0000 R CNN
-F 2 "LEDs:LED_0603_HandSoldering" H 7500 2200 50  0001 C CNN
+F 2 "LEDs:LED_0805_HandSoldering" H 7500 2200 50  0001 C CNN
 F 3 "~" H 7500 2200 50  0001 C CNN
 	1    7500 2200
@@
 F 0 "R12" V 7293 2500 50  0000 C CNN
 F 1 "1K" V 7384 2500 50  0000 C CNN
-F 2 "Resistor_SMD:R_0603_1608Metric_Pad1.05x0.95mm_HandSolder" V 7430 2500 50  0001 C CNN
+F 2 "Resistors_SMD:R_0805_HandSoldering" V 7430 2500 50  0001 C CNN
 F 3 "~" H 7500 2500 50  0001 C CNN
 	1    7500 2500
@@
 F 0 "R13" V 7593 3900 50  0000 C CNN
 F 1 "1K" V 7684 3900 50  0000 C CNN
-F 2 "Resistor_SMD:R_0603_1608Metric_Pad1.05x0.95mm_HandSolder" V 7730 3900 50  0001 C CNN
+F 2 "Resistors_SMD:R_0805_HandSoldering" V 7730 3900 50  0001 C CNN
 F 3 "~" H 7800 3900 50  0001 C CNN
 	1    7800 3900
@@
 F 0 "D7" V 8288 3033 50  0000 R CNN
 F 1 "LED" V 8197 3033 50  0000 R CNN
-F 2 "LEDs:LED_0603_HandSoldering" H 8250 3150 50  0001 C CNN
+F 2 "LEDs:LED_0805_HandSoldering" H 8250 3150 50  0001 C CNN
 F 3 "~" H 8250 3150 50  0001 C CNN
 	1    8250 3150
@@
 F 0 "R14" V 8043 3450 50  0000 C CNN
 F 1 "1K" V 8134 3450 50  0000 C CNN
-F 2 "Resistor_SMD:R_0603_1608Metric_Pad1.05x0.95mm_HandSolder" V 8180 3450 50  0001 C CNN
+F 2 "Resistors_SMD:R_0805_HandSoldering" V 8180 3450 50  0001 C CNN
 F 3 "~" H 8250 3450 50  0001 C CNN
 	1    8250 3450
@@
 F 0 "R15" V 8393 4800 50  0000 C CNN
 F 1 "1K" V 8484 4800 50  0000 C CNN
-F 2 "Resistor_SMD:R_0603_1608Metric_Pad1.05x0.95mm_HandSolder" V 8530 4800 50  0001 C CNN
+F 2 "Resistors_SMD:R_0805_HandSoldering" V 8530 4800 50  0001 C CNN
 F 3 "~" H 8600 4800 50  0001 C CNN
 	1    8600 4800
@@
 F 0 "D8" V 9088 3933 50  0000 R CNN
 F 1 "LED" V 8997 3933 50  0000 R CNN
-F 2 "LEDs:LED_0603_HandSoldering" H 9050 4050 50  0001 C CNN
+F 2 "LEDs:LED_0805_HandSoldering" H 9050 4050 50  0001 C CNN
 F 3 "~" H 9050 4050 50  0001 C CNN
 	1    9050 4050
@@
 F 0 "R16" V 8843 4350 50  0000 C CNN
 F 1 "1K" V 8934 4350 50  0000 C CNN
-F 2 "Resistor_SMD:R_0603_1608Metric_Pad1.05x0.95mm_HandSolder" V 8980 4350 50  0001 C CNN
+F 2 "Resistors_SMD:R_0805_HandSoldering" V 8980 4350 50  0001 C CNN
 F 3 "~" H 9050 4350 50  0001 C CNN
 	1    9050 4350
