File: Projects/Sonoff_4Ch_Switch/Sonoff_4ch_switch-Rev A2.sch (KiCad schematic (older format))
At the start: 23 parts, among them J1 Barrel_Jack_Switch, J5 Conn_01x03_Male, U1 AP1117-50, U2 Wemos_D1_Mini_wide

Commit message: On to rev A2 of the 4 ch switch....
Parts:
- added MH1, MH2, MH3, MH4: MountingHole, Mounting_Holes:MountingHole_3mm_Pad, symbol Mechanical:MountingHole
- added TP3: GND, Measurement_Points:Measurement_Point_Round-SMD-Pad_Small, symbol Connector:TestPoint
- D9: footprint LEDs:LED_0603_HandSoldering -> LEDs:LED_0805_HandSoldering
- R17, R18, R19, R20, R21, R22: footprint Resistor_SMD:R_0603_1608Metric_Pad1.05x0.95mm_HandSolder -> Resistors_SMD:R_0805_HandSoldering
- TP1: footprint TestPoint:TestPoint_Pad_D2.0mm -> Measurement_Points:Measurement_Point_Round-SMD-Pad_Small
- U2: footprint (none) -> My_Component_Footprints:Wemos_D1_mini_board-flipped
- gave numbers to parts that had none: 4
Connections:
- wire segments 80 -> 81
Other:
- note added: "Design notes for rev A2:\n1. Add a GND TP, with a pin(?) - Done\n2. No Reverse polarity protection\n3. Do away with the Regulator? Run it from 5V Power bricks?\n4. Redesign the layout with 0805 components! (0603 too small) - Done\n5. If keeping the regulator, re-engineer the copper pad for 5V, needs to be larger.\n6. Sort out the switch order! - DONE\n"
