File: Projects/Sonoff_4Ch_Switch/Sonoff_4ch_switch.sch (KiCad schematic (older format))
At the start: 19 parts, among them J1 Barrel_Jack_Switch, J5 Conn_01x03_Male, U1 AP1117-50, U2 Wemos_D1_Mini_wide

Commit message: On to rev A2 of the 4 ch switch....
Parts:
- added F1: Fuse 5A, Fuse_Holders_and_Fuses:Fuseholder5x20_horiz_SemiClosed_Casing10x25mm, symbol Device:Fuse
- added J2: Live, TerminalBlock_RND:TerminalBlock_RND_205-00004_1x05_P5.00mm_Horizontal, symbol Connector:Screw_Terminal_01x05
- added J3: Neutrals, TerminalBlock_RND:TerminalBlock_RND_205-00004_1x05_P5.00mm_Horizontal, symbol Connector:Screw_Terminal_01x05
- added J4: Earths, TerminalBlock_RND:TerminalBlock_RND_205-00004_1x05_P5.00mm_Horizontal, symbol Connector:Screw_Terminal_01x05
- added TP3: GND, TestPoint:TestPoint_Pad_D2.0mm, symbol Connector:TestPoint
- R17, R18, R19, R20, R21, R22: footprint Resistor_SMD:R_0603_1608Metric_Pad1.05x0.95mm_HandSolder -> Resistors_SMD:R_0805_HandSoldering
Connections:
- net labels added: AC, Earth, L1, L2, L3, L4, LineIN, Neutral
- wire segments 52 -> 81
Other:
- note added: "Design notes:\n1. Add a GND TP, with a pin(?)\n2. No Reverse polarity protection\n3. Do away with the Regulator? Run it from 5V Power bricks?\n4. Redesign the layout with 0805 components! (0603 too small)\n5. If keeping the regulator, re-engineer the copper pad for 5V, needs to be larger.\n6. Sort out the switch order!\n"
- note added: "Mains Terminal Blocks"
- moved on the sheet: U1
