File: Projects/Tasmota 2 CH Switch/Relays.sch (KiCad schematic (older format))
At the start: 36 parts, among them K1 G5LE-1, K2 G5LE-1, K3 G5LE-1, K4 G5LE-1, Q1 2N7002, Q2 2N7002, Q3 2N7002, Q4 2N7002, Q5 2N7002, Q6 2N7002, Q7 2N7002, Q8 2N7002

Commit message: Created new 2Ch Tasmota Switch
Parts:
- renumbered D1 to D?, D2 to D?, D3 to D?, D4 to D?, D5 to D?, D6 to D?, D7 to D?, D8 to D?, K1 to K?, K2 to K?, K3 to K?, K4 to K?, Q1 to Q?, Q2 to Q?, Q3 to Q?, Q4 to Q?, Q5 to Q?, Q6 to Q?, Q7 to Q?, Q8 to Q?, R1 to R?, R2 to R?, R3 to R?, R4 to R?, R5 to R?, R6 to R?, R7 to R?, R8 to R?, R9 to R?, R10 to R?, R11 to R?, R12 to R?, R13 to R?, R14 to R?, R15 to R?, R16 to R?
