File: Projects/Sonoff_2ch_switch Rev A1/Relays.sch (KiCad schematic (older format))
At the start: 36 parts

Commit message: SOrted out 2Ch layout, condensed into a single SCH sheet
Parts:
- removed D? (x2): 1N4148, Diodes_SMD:D_SOD-123, symbol Device:D
- removed D? (x2): LED, LEDs:LED_0805_HandSoldering, symbol Device:LED
- removed K? (x2): G5LE-1, Relay_THT:Relay_SPDT_Omron-G5LE-1, symbol Relay:G5LE-1
- removed Q? (x4): 2N7002, Package_TO_SOT_SMD:SOT-23, symbol Transistor_FET:2N7002
- removed R? (x6): 1K, Resistors_SMD:R_0805_HandSoldering, symbol Device:R
- removed R? (x2): 10K, Resistors_SMD:R_0805_HandSoldering, symbol Device:R
Connections:
- net labels removed: L3, L4, Relay3, Relay4
- wire segments 92 -> 46
- no-connect marks 5 -> 3
