File: Projects/Fibre Tester/Fibre Tester.sch (KiCad schematic (older format))
At the start: 9 parts, among them IC1 NE555

Commit message: Updated Fibre Tester project
Parts:
- removed S1: JS202011SCQN, NetTie:NetTie-4_SMD_Pad2.0mm, symbol dk_Slide-Switches:JS202011SCQN
- added H1, H2, H3, H4: MountingHole, MountingHole:MountingHole_2.5mm, symbol Mechanical:MountingHole
- added SW1: SW_SPDT, My_Component_Footprints:SW_Slide_angle_SPDT_TB, symbol Switch:SW_SPDT
- BT1: footprint Jumper:SolderJumper-2_P1.3mm_Open_Pad1.0x1.5mm -> Connector_PinSocket_2.54mm:PinSocket_1x02_P2.54mm_Vertical
- R1: renamed from R3; footprint Resistor_THT:R_Axial_DIN0309_L9.0mm_D3.2mm_P12.70mm_Horizontal -> Resistor_THT:R_Axial_DIN0207_L6.3mm_D2.5mm_P10.16mm_Horizontal
- R2: renamed from R1; footprint Resistor_THT:R_Axial_DIN0309_L9.0mm_D3.2mm_P12.70mm_Horizontal -> Resistor_THT:R_Axial_DIN0207_L6.3mm_D2.5mm_P10.16mm_Horizontal
- R3: renamed from R2; footprint Resistor_THT:R_Axial_DIN0309_L9.0mm_D3.2mm_P12.70mm_Horizontal -> Resistor_THT:R_Axial_DIN0207_L6.3mm_D2.5mm_P10.16mm_Horizontal
Connections:
- net VCC: now also D1.2 (A), SW1.3 (C)
- net at BT1.1 (+): now also SW1.2 (B)
- no-connect marks 6 -> 3
Changed lines of the file:
@@
 $EndComp
 $Comp
-L Fibre-Tester-rescue:R0207_10-Fibre_Tester-eagle-import R1
+L Fibre-Tester-rescue:R0207_10-Fibre_Tester-eagle-import R2
 U 1 0 A4A47D12
 P 5600 3100
-F 0 "R1" H 5450 3159 59  0000 L BNN
+F 0 "R2" H 5450 3159 59  0000 L BNN
 F 1 "220" H 5450 2970 59  0000 L BNN
-F 2 "Resistor_THT:R_Axial_DIN0309_L9.0mm_D3.2mm_P12.70mm_Horizontal" H 5600 3100 50  0001 C CNN
+F 2 "Resistor_THT:R_Axial_DIN0207_L6.3mm_D2.5mm_P10.16mm_Horizontal" H 5600 3100 50  0001 C CNN
 F 3 "" H 5600 3100 50  0001 C CNN
 	1    5600 3100
@@
 $EndComp
 $Comp
-L Fibre-Tester-rescue:R0207_10-Fibre_Tester-eagle-import R2
+L Fibre-Tester-rescue:R0207_10-Fibre_Tester-eagle-import R3
 U 1 0 759C9AAF
 P 5600 3700
-F 0 "R2" H 5450 3759 59  0000 L BNN
+F 0 "R3" H 5450 3759 59  0000 L BNN
 F 1 "220" H 5450 3570 59  0000 L BNN
-F 2 "Resistor_THT:R_Axial_DIN0309_L9.0mm_D3.2mm_P12.70mm_Horizontal" H 5600 3700 50  0001 C CNN
+F 2 "Resistor_THT:R_Axial_DIN0207_L6.3mm_D2.5mm_P10.16mm_Horizontal" H 5600 3700 50  0001 C CNN
 F 3 "" H 5600 3700 50  0001 C CNN
 	1    5600 3700
@@
 $EndComp
 $Comp
-L Fibre-Tester-rescue:R0207_10-Fibre_Tester-eagle-import R3
+L Fibre-Tester-rescue:R0207_10-Fibre_Tester-eagle-import R1
 U 1 0 7FD4C25A
 P 3700 2800
-F 0 "R3" H 3550 2859 59  0000 L BNN
+F 0 "R1" H 3550 2859 59  0000 L BNN
 F 1 "47k" H 3550 2670 59  0000 L BNN
-F 2 "Resistor_THT:R_Axial_DIN0309_L9.0mm_D3.2mm_P12.70mm_Horizontal" H 3700 2800 50  0001 C CNN
+F 2 "Resistor_THT:R_Axial_DIN0207_L6.3mm_D2.5mm_P10.16mm_Horizontal" H 3700 2800 50  0001 C CNN
 F 3 "" H 3700 2800 50  0001 C CNN
 	1    3700 2800
@@
 $EndComp
 $Comp
-L Fibre-Tester-rescue:GND-Fibre_Tester-eagle-import #GND01
+L Fibre-Tester-rescue:GND-Fibre_Tester-eagle-import #GND02
 U 1 0 8DA2BB24
 P 3700 4600
-F 0 "#GND01" H 3700 4600 50  0001 C CNN
+F 0 "#GND02" H 3700 4600 50  0001 C CNN
 F 1 "GND" H 3600 4500 59  0000 L BNN
 F 2 "" H 3700 4600 50  0001 C CNN
@@
 $EndComp
 $Comp
-L power:VCC #PWR01
+L power:VCC #PWR02
 U 1 1 5CBFF78D
 P 4950 3150
-F 0 "#PWR01" H 4950 3000 50  0001 C CNN
+F 0 "#PWR02" H 4950 3000 50  0001 C CNN
 F 1 "VCC" H 4967 3323 50  0000 C CNN
 F 2 "" H 4950 3150 50  0001 C CNN
 F 3 "" H 4950 3150 50  0001 C CNN
 	1    4950 3150
-	1    0    0    -1
-$EndComp
-$Comp
-L dk_Slide-Switches:JS202011SCQN S1
-U 1 1 5CBFFF09
-P 4300 1800
-F 0 "S1" H 4300 2283 50  0000 C CNN
-F 1 "JS202011SCQN" H 4300 2192 50  0000 C CNN
-F 2 "NetTie:NetTie-4_SMD_Pad2.0mm" H 4500 2000 50  0001 L CNN
-F 3 "https://www.ckswitches.com/media/1422/js.pdf" H 4500 2100 60  0001 L CNN
-F 4 "401-2002-1-ND" H 4500 2200 60  0001 L CNN "Digi-Key_PN"
-F 5 "JS202011SCQN" H 4500 2300 60  0001 L CNN "MPN"
-F 6 "Switches" H 4500 2400 60  0001 L CNN "Category"
-F 7 "Slide Switches" H 4500 2500 60  0001 L CNN "Family"
-F 8 "https://www.ckswitches.com/media/1422/js.pdf" H 4500 2600 60  0001 L CNN "DK_Datasheet_Link"
-F 9 "/product-detail/en/c-k/JS202011SCQN/401-2002-1-ND/1640098" H 4500 2700 60  0001 L CNN "DK_Detail_Page"
-F 10 "SWITCH SLIDE DPDT 300MA 6V" H 4500 2800 60  0001 L CNN "Description"
-F 11 "C&K" H 4500 2900 60  0001 L CNN "Manufacturer"
-F 12 "Active" H 4500 3000 60  0001 L CNN "Status"
-	1    4300 1800
-	1    0    0    -1
-$EndComp
-Wire Wire Line
-	4500 2100 5600 2100
-$Comp
-L Device:Battery_Cell BT1
-U 1 1 5CC00832
-P 3100 2200
-F 0 "BT1" H 3218 2296 50  0000 L CNN
-F 1 "Battery_Cell" H 3218 2205 50  0000 L CNN
-F 2 "Jumper:SolderJumper-2_P1.3mm_Open_Pad1.0x1.5mm" V 3100 2260 50  0001 C CNN
-F 3 "~" V 3100 2260 50  0001 C CNN
-	1    3100 2200
 	1    0    0    -1
 $EndComp
@@
 $EndComp
 Wire Wire Line
-	4100 2000 3100 2000
-Wire Wire Line
 	4950 3200 4950 3150
 Wire Wire Line
@@
 Wire Wire Line
 	4700 3800 4900 3800
-NoConn ~ 4500 1500
-NoConn ~ 4500 1700
-NoConn ~ 4100 1600
-NoConn ~ 4500 1900
-$Comp
-L Fibre-Tester-rescue:GND-Fibre_Tester-eagle-import #GND0101
+$Comp
+L Fibre-Tester-rescue:GND-Fibre_Tester-eagle-import #GND01
 U 1 1 5CC02BEF
-P 3100 2400
-F 0 "#GND0101" H 3100 2400 50  0001 C CNN
-F 1 "GND" H 3100 2279 59  0000 C CNN
-F 2 "" H 3100 2400 50  0001 C CNN
-F 3 "" H 3100 2400 50  0001 C CNN
-	1    3100 2400
+P 2800 2500
+F 0 "#GND01" H 2800 2500 50  0001 C CNN
+F 1 "GND" H 2800 2379 59  0000 C CNN
+F 2 "" H 2800 2500 50  0001 C CNN
+F 3 "" H 2800 2500 50  0001 C CNN
+	1    2800 2500
 	1    0    0    -1
 $EndComp
@@
 	1    0    0    -1
 $EndComp
+$Comp
+L Switch:SW_SPDT SW1
+U 1 1 5D034C9B
+P 4150 2000
+F 0 "SW1" H 4150 2285 50  0000 C CNN
+F 1 "SW_SPDT" H 4150 2194 50  0000 C CNN
+F 2 "My_Component_Footprints:SW_Slide_angle_SPDT_TB" H 4150 2000 50  0001 C CNN
+F 3 "~" H 4150 2000 50  0001 C CNN
+	1    4150 2000
+	1    0    0    -1
+$EndComp
+Wire Wire Line
+	4350 2100 4800 2100
+Wire Wire Line
+	2800 2000 2800 2100
+Wire Wire Line
+	2800 2000 3950 2000
+NoConn ~ 4350 1900
+$Comp
+L power:VCC #PWR01
+U 1 1 5D036325
+P 4800 2100
+F 0 "#PWR01" H 4800 1950 50  0001 C CNN
+F 1 "VCC" H 4817 2273 50  0000 C CNN
+F 2 "" H 4800 2100 50  0001 C CNN
+F 3 "" H 4800 2100 50  0001 C CNN
+	1    4800 2100
+	1    0    0    -1
+$EndComp
+Connection ~ 4800 2100
+Wire Wire Line
+	4800 2100 5600 2100
+$Comp
+L Mechanical:MountingHole H4
+U 1 1 5D03D188
+P 800 2650
+F 0 "H4" H 900 2696 50  0000 L CNN
+F 1 "MountingHole" H 900 2605 50  0000 L CNN
+F 2 "MountingHole:MountingHole_2.5mm" H 800 2650 50  0001 C CNN
+F 3 "~" H 800 2650 50  0001 C CNN
+	1    800  2650
+	1    0    0    -1
+$EndComp
+$Comp
+L Mechanical:MountingHole H3
+U 1 1 5D03CE9F
+P 800 2450
+F 0 "H3" H 900 2496 50  0000 L CNN
+F 1 "MountingHole" H 900 2405 50  0000 L CNN
+F 2 "MountingHole:MountingHole_2.5mm" H 800 2450 50  0001 C CNN
+F 3 "~" H 800 2450 50  0001 C CNN
+	1    800  2450
+	1    0    0    -1
+$EndComp
+$Comp
+L Mechanical:MountingHole H2
+U 1 1 5D03CAF1
+P 800 2250
+F 0 "H2" H 900 2296 50  0000 L CNN
+F 1 "MountingHole" H 900 2205 50  0000 L CNN
+F 2 "MountingHole:MountingHole_2.5mm" H 800 2250 50  0001 C CNN
+F 3 "~" H 800 2250 50  0001 C CNN
+	1    800  2250
+	1    0    0    -1
+$EndComp
+$Comp
+L Mechanical:MountingHole H1
+U 1 1 5D03C183
+P 800 2050
+F 0 "H1" H 900 2096 50  0000 L CNN
+F 1 "MountingHole" H 900 2005 50  0000 L CNN
+F 2 "MountingHole:MountingHole_2.5mm" H 800 2050 50  0001 C CNN
+F 3 "~" H 800 2050 50  0001 C CNN
+	1    800  2050
+	1    0    0    -1
+$EndComp
+$Comp
+L Device:Battery_Cell BT1
+U 1 1 5D04C074
+P 2800 2300
+F 0 "BT1" H 2918 2396 50  0000 L CNN
+F 1 "Battery_Cell" H 2918 2305 50  0000 L CNN
+F 2 "Connector_PinSocket_2.54mm:PinSocket_1x02_P2.54mm_Vertical" V 2800 2360 50  0001 C CNN
+F 3 "~" V 2800 2360 50  0001 C CNN
+	1    2800 2300
+	1    0    0    -1
+$EndComp
